File: board/HM-10 Breakout.brd (EAGLE design)
At the start: 24 x 33.7 mm, 20 parts, among them U1 V_REG_LDOSMD, U2 HM-10

Commit message: Update images
Parts:
- U$2: device SparkFun-Aesthetics:OSHW-LOGO-M -> SparkFun-Aesthetics:OSHW-LOGO-S
- moved U$1 2.70 mm to (12.0, 4.65)
- moved U$2 0.21 mm to (11.8, 30.6)
Changed lines of the file:
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@@
 <text x="20.80539375" y="32.019790625" size="1.27" layer="26" font="vector" rot="MR0" align="center-left">GND</text>
 <text x="14.55" y="20.25" size="0.6096" layer="25" rot="R90">v1.1</text>
-<text x="14.55" y="8.85" size="0.6096" layer="25" rot="R90">Breakout Board</text>
+<text x="14.55" y="8.85" size="0.8128" layer="25" rot="R90">Breakout Board</text>
 <text x="20.886" y="14.202" size="1.27" layer="26" font="vector" rot="MR0" align="center-left">DC</text>
 <text x="20.886" y="11.652" size="1.27" layer="26" font="vector" rot="MR0" align="center-left">DD</text>
-<text x="12" y="5.1" size="0.8128" layer="26" font="vector" rot="MR0" align="bottom-center">HM-10 Breakout</text>
-<text x="16.95" y="4.2" size="0.6096" layer="26" font="vector" rot="MR0">Nick Walker</text>
-<text x="7.05" y="4.2" size="0.6096" layer="26" font="vector" rot="MR0" align="bottom-right">v1.1</text>
+<text x="11.85" y="1.8" size="0.8128" layer="26" font="vector" rot="MR0" align="bottom-center">HM-10 Breakout</text>
+<text x="16.8" y="0.9" size="0.6096" layer="26" font="vector" rot="MR0">Nick Walker</text>
+<text x="6.9" y="0.9" size="0.6096" layer="26" font="vector" rot="MR0" align="bottom-right">v1.1</text>
 </plain>
 <attributes>
@@
 <element name="C2" library="resistor" package="C0805K" value="1uF" x="9.4347375" y="16.303146875" smashed="yes" rot="MR270"/>
 <element name="U2" library="HM-10_BLE" package="HM-10" value="HM-10" x="12" y="13.95" rot="R180"/>
-<element name="U$2" library="SparkFun-Aesthetics" package="OSHW-LOGO-M" value="" x="12" y="30.75" smashed="yes"/>
-<element name="U$1" library="SparkFun-Aesthetics" package="OSHW-LOGO-S" value="" x="12" y="1.95" smashed="yes" rot="MR0"/>
+<element name="U$1" library="SparkFun-Aesthetics" package="OSHW-LOGO-S" value="" x="12" y="4.65" smashed="yes" rot="MR0"/>
+<element name="U$2" library="SparkFun-Aesthetics" package="OSHW-LOGO-S" value="" x="11.85" y="30.6"/>
 </elements>
 <signals>
